File: board/cells.kicad_sch (KiCad schematic)
At the start: 3 parts

Commit message: initial
Parts:
- BT1, BT2: value BHAA-3-G -> (none); footprint BAT_BHAA-3-G -> (none)
- R1: value 0R -> (none); footprint Resistor_SMD:R_0603_1608Metric -> (none)
Changed lines of the file:
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@@
       (effects (font (size 1.27 1.27)) (justify right))
     )
-    (property "Value" "BHAA-3-G" (id 1) (at 153.67 86.9951 90)
+    (property "Value" "" (id 1) (at 153.67 86.9951 90)
       (effects (font (size 1.27 1.27)) (justify right))
     )
-    (property "Footprint" "BAT_BHAA-3-G" (id 2) (at 157.48 88.9 0)
+    (property "Footprint" "" (id 2) (at 157.48 88.9 0)
       (effects (font (size 1.27 1.27)) (justify bottom) hide)
     )
@@
       (effects (font (size 1.27 1.27)) (justify right))
     )
-    (property "Value" "BHAA-3-G" (id 1) (at 153.67 104.7751 90)
+    (property "Value" "" (id 1) (at 153.67 104.7751 90)
       (effects (font (size 1.27 1.27)) (justify right))
     )
-    (property "Footprint" "BAT_BHAA-3-G" (id 2) (at 157.48 106.68 0)
+    (property "Footprint" "" (id 2) (at 157.48 106.68 0)
       (effects (font (size 1.27 1.27)) (justify bottom) hide)
     )
@@
       (effects (font (size 1.27 1.27)) (justify left))
     )
-    (property "Value" "0R" (id 1) (at 160.02 120.6499 0)
+    (property "Value" "" (id 1) (at 160.02 120.6499 0)
       (effects (font (size 1.27 1.27)) (justify left))
     )
-    (property "Footprint" "Resistor_SMD:R_0603_1608Metric" (id 2) (at 157.48 119.38 0)
+    (property "Footprint" "" (id 2) (at 157.48 119.38 0)
       (effects (font (size 1.27 1.27)) hide)
     )
